File: hardware/pcdu/rev1_4/rev_1_4.sch (EAGLE design)
At the start: 17 parts, among them IC1 74HC595N, X1 KUSBVX, X10 22-23-2041, X11 22-23-2041, X2 KUSBVX, X3 KUSBVX, X4 KUSBVX, X5 KUSBVX, X6 KUSBVX, X7 KUSBVX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

Commit message: Started work on rev1_4 board
Parts:
- removed X1, X2, X3, X4, X5, X6, X7, X8: KUSBVX, con-kycon:KUSBVX
- added U$5, U$6, U$7, U$8: USB2V, USB2V:USB2V
- X9: value (none) -> 5v
Connections:
- removed net N$10: U$1.D2, X2.4, X2.S1, X2.S2
- removed net N$11: U$2.D1, X3.4, X3.S1, X3.S2
- removed net N$12: U$2.D2, X4.4, X4.S1, X4.S2
- removed net N$13: U$3.D1, X5.4, X5.S1, X5.S2
- removed net N$14: U$3.D2, X6.4, X6.S1, X6.S2
- removed net N$15: U$4.D1, X7.4, X7.S1, X7.S2
- removed net N$16: U$4.D2, X8.4, X8.S1, X8.S2
- removed net N$9: U$1.D1, X1.4, X1.S1, X1.S2
- new net N$1: U$1.D1, U$5.G2, U$5.GL2, U$5.GR2
- new net N$2: U$1.D2, U$5.G1, U$5.GL1, U$5.GR1
- new net N$3: U$2.D1, U$6.G2, U$6.GL2, U$6.GR2
- new net N$4: U$2.D2, U$6.G1, U$6.GL1, U$6.GR1
- new net N$5: U$3.D1, U$7.G2, U$7.GL2, U$7.GR2
- new net N$6: U$3.D2, U$7.G1, U$7.GL1, U$7.GR1
- new net N$7: U$4.D1, U$8.G2, U$8.GL2, U$8.GR2
- new net N$8: U$4.D2, U$8.G1, U$8.GL1, U$8.GR1
- net VCC: now also U$5.V1, U$5.V2, U$6.V1, U$6.V2, U$7.V1, U$7.V2, U$8.V1, U$8.V2; no longer X1.1, X2.1, X3.1, X4.1, X5.1, X6.1, X7.1, X8.1
Other:
- moved on the sheet: U$1
