File: hardware/pcdu/rev1_6/rev1_6.sch (EAGLE design)
At the start: 17 parts, among them IC1 74HC595N, X1 MUSBV, X2 MUSBV, X3 MUSBV, X4 MUSBV, X7 22-23-2041, X8 22-23-2041

Commit message: Updated PDU board, removed screw terminal
Parts:
- IC1: value 74HC595N -> 74HC595D; device 74xx-eu:74HC595N -> 74xx-eu:74HC595D
Other:
- moved on the sheet: IC1P
Changed lines of the file:
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@@
 </classes>
 <parts>
-<part name="IC1" library="74xx-eu" deviceset="74*595" device="N" technology="HC"/>
 <part name="U$1" library="FDC6305N" deviceset="FDC6305N" device=""/>
 <part name="U$2" library="FDC6305N" deviceset="FDC6305N" device=""/>
@@
 <part name="R3" library="eagle-ltspice" deviceset="R" device="R1005"/>
 <part name="R4" library="eagle-ltspice" deviceset="R" device="R1005"/>
+<part name="IC1" library="74xx-eu" deviceset="74*595" device="D" technology="HC"/>
 </parts>
 <sheets>
@@
 </plain>
 <instances>
-<instance part="IC1" gate="A" x="81.28" y="12.7" rot="R90"/>
 <instance part="U$1" gate="G$1" x="50.8" y="50.8" rot="R270"/>
 <instance part="U$2" gate="G$1" x="116.84" y="50.8" rot="R270"/>
@@
 <instance part="X8" gate="-3" x="33.02" y="-33.02" rot="MR0"/>
 <instance part="X8" gate="-4" x="33.02" y="-35.56" rot="MR0"/>
-<instance part="IC1" gate="P" x="60.96" y="12.7"/>
 <instance part="X1" gate="G$1" x="35.56" y="76.2"/>
 <instance part="X2" gate="G$1" x="66.04" y="76.2"/>
@@
 <instance part="R3" gate="G$1" x="86.36" y="43.18" rot="R90"/>
 <instance part="R4" gate="G$1" x="93.98" y="43.18" rot="R90"/>
+<instance part="IC1" gate="A" x="81.28" y="12.7" rot="R90"/>
+<instance part="IC1" gate="P" x="53.34" y="10.16"/>
 </instances>
 <busses>
@@
 <net name="VCC" class="0">
 <segment>
-<pinref part="IC1" gate="P" pin="VCC"/>
-<wire x1="60.96" y1="20.32" x2="60.96" y2="22.86" width="0.1524" layer="91"/>
-<label x="55.88" y="20.32" size="1.778" layer="95"/>
-</segment>
-<segment>
-<pinref part="IC1" gate="A" pin="SCL"/>
 <wire x1="78.74" y1="0" x2="78.74" y2="-2.54" width="0.1524" layer="91"/>
 <label x="78.74" y="-5.08" size="1.778" layer="95"/>
+<pinref part="IC1" gate="A" pin="SCL"/>
 </segment>
 <segment>
@@
 <label x="81.28" y="58.42" size="1.778" layer="95"/>
 </segment>
+<segment>
+<pinref part="IC1" gate="P" pin="VCC"/>
+<wire x1="53.34" y1="17.78" x2="53.34" y2="20.32" width="0.1524" layer="91"/>
+<label x="48.26" y="20.32" size="1.778" layer="95"/>
+</segment>
 </net>
 <net name="GND" class="0">
@@
 </segment>
 <segment>
-<pinref part="IC1" gate="P" pin="GND"/>
-<wire x1="60.96" y1="5.08" x2="60.96" y2="2.54" width="0.1524" layer="91"/>
-<label x="55.88" y="2.54" size="1.778" layer="95"/>
-</segment>
-<segment>
-<pinref part="IC1" gate="A" pin="G"/>
 <wire x1="93.98" y1="0" x2="93.98" y2="-2.54" width="0.1524" layer="91"/>
 <label x="93.98" y="-2.54" size="1.778" layer="95"/>
+<pinref part="IC1" gate="A" pin="G"/>
 </segment>
 <segment>
@@
 <label x="111.76" y="63.5" size="1.778" layer="95"/>
 </segment>
+<segment>
+<pinref part="IC1" gate="P" pin="GND"/>
+<wire x1="53.34" y1="2.54" x2="53.34" y2="0" width="0.1524" layer="91"/>
+<label x="48.26" y="0" size="1.778" layer="95"/>
+</segment>
 </net>
 <net name="N$1" class="0">
 <segment>
-<pinref part="IC1" gate="A" pin="QA"/>
 <pinref part="U$1" gate="G$1" pin="G1"/>
 <wire x1="71.12" y1="25.4" x2="48.26" y2="25.4" width="0.1524" layer="91"/>
 <wire x1="48.26" y1="25.4" x2="48.26" y2="38.1" width="0.1524" layer="91"/>
+<pinref part="IC1" gate="A" pin="QA"/>
 </segment>
 </net>
 <net name="N$2" class="0">
 <segment>
-<pinref part="IC1" gate="A" pin="QB"/>
 <wire x1="73.66" y1="25.4" x2="73.66" y2="27.94" width="0.1524" layer="91"/>
 <pinref part="U$1" gate="G$1" pin="G2"/>
 <wire x1="73.66" y1="27.94" x2="53.34" y2="27.94" width="0.1524" layer="91"/>
 <wire x1="53.34" y1="27.94" x2="53.34" y2="38.1" width="0.1524" layer="91"/>
+<pinref part="IC1" gate="A" pin="QB"/>
 </segment>
 </net>
 <net name="N$3" class="0">
 <segment>
-<pinref part="IC1" gate="A" pin="QC"/>
 <wire x1="76.2" y1="25.4" x2="76.2" y2="30.48" width="0.1524" layer="91"/>
 <pinref part="U$2" gate="G$1" pin="G1"/>
 <wire x1="76.2" y1="30.48" x2="114.3" y2="30.48" width="0.1524" layer="91"/>
 <wire x1="114.3" y1="30.48" x2="114.3" y2="38.1" width="0.1524" layer="91"/>
+<pinref part="IC1" gate="A" pin="QC"/>
 </segment>
 </net>
 <net name="N$4" class="0">
 <segment>
-<pinref part="IC1" gate="A" pin="QD"/>
 <wire x1="78.74" y1="25.4" x2="78.74" y2="27.94" width="0.1524" layer="91"/>
 <pinref part="U$2" gate="G$1" pin="G2"/>
 <wire x1="78.74" y1="27.94" x2="119.38" y2="27.94" width="0.1524" layer="91"/>
 <wire x1="119.38" y1="27.94" x2="119.38" y2="38.1" width="0.1524" layer="91"/>
+<pinref part="IC1" gate="A" pin="QD"/>
 </segment>
 </net>
 <net name="SOUT" class="0">
 <segment>
-<pinref part="IC1" gate="A" pin="QH*"/>
 <wire x1="93.98" y1="25.4" x2="96.52" y2="25.4" width="0.1524" layer="91"/>
 <label x="96.52" y="25.4" size="1.778" layer="95"/>
+<pinref part="IC1" gate="A" pin="QH*"/>
 </segment>
 <segment>
@@
 </segment>
 <segment>
-<pinref part="IC1" gate="A" pin="SER"/>
 <wire x1="71.12" y1="0" x2="71.12" y2="-2.54" width="0.1524" layer="91"/>
 <label x="66.04" y="-2.54" size="1.778" layer="95"/>
+<pinref part="IC1" gate="A" pin="SER"/>
 </segment>
 </net>
@@
 </segment>
 <segment>
-<pinref part="IC1" gate="A" pin="SCK"/>
 <wire x1="76.2" y1="0" x2="76.2" y2="-2.54" width="0.1524" layer="91"/>
 <label x="73.66" y="-5.08" size="1.778" layer="95"/>
+<pinref part="IC1" gate="A" pin="SCK"/>
 </segment>
 </net>
@@
 </segment>
 <segment>
-<pinref part="IC1" gate="A" pin="RCK"/>
 <wire x1="83.82" y1="0" x2="83.82" y2="-2.54" width="0.1524" layer="91"/>
 <label x="83.82" y="-2.54" size="1.778" layer="95"/>
+<pinref part="IC1" gate="A" pin="RCK"/>
 </segment>
 </net>
@@
 <net name="N$13" class="0">
 <segment>
-<pinref part="IC1" gate="A" pin="QE"/>
 <wire x1="81.28" y1="33.02" x2="81.28" y2="25.4" width="0.1524" layer="91"/>
 <wire x1="81.28" y1="33.02" x2="71.12" y2="33.02" width="0.1524" layer="91"/>
 <wire x1="71.12" y1="33.02" x2="71.12" y2="38.1" width="0.1524" layer="91"/>
 <pinref part="R1" gate="G$1" pin="1"/>
+<pinref part="IC1" gate="A" pin="QE"/>
 </segment>
 </net>
 <net name="N$14" class="0">
 <segment>
-<pinref part="IC1" gate="A" pin="QF"/>
 <wire x1="83.82" y1="25.4" x2="83.82" y2="35.56" width="0.1524" layer="91"/>
 <wire x1="83.82" y1="35.56" x2="78.74" y2="35.56" width="0.1524" layer="91"/>
 <wire x1="78.74" y1="35.56" x2="78.74" y2="38.1" width="0.1524" layer="91"/>
 <pinref part="R2" gate="G$1" pin="1"/>
+<pinref part="IC1" gate="A" pin="QF"/>
 </segment>
 </net>
 <net name="N$15" class="0">
 <segment>
-<pinref part="IC1" gate="A" pin="QG"/>
 <wire x1="86.36" y1="25.4" x2="86.36" y2="38.1" width="0.1524" layer="91"/>
 <pinref part="R3" gate="G$1" pin="1"/>
+<pinref part="IC1" gate="A" pin="QG"/>
 </segment>
 </net>
 <net name="N$16" class="0">
 <segment>
-<pinref part="IC1" gate="A" pin="QH"/>
 <wire x1="88.9" y1="25.4" x2="88.9" y2="35.56" width="0.1524" layer="91"/>
 <wire x1="88.9" y1="35.56" x2="93.98" y2="35.56" width="0.1524" layer="91"/>
 <wire x1="93.98" y1="35.56" x2="93.98" y2="38.1" width="0.1524" layer="91"/>
 <pinref part="R4" gate="G$1" pin="1"/>
-</segment>
-</net>
+<pinref part="IC1" gate="A" pin="QH"/>
+</segment>
+</net>
